File: Tode-BIOPH/kicad/IO-ACCESS/SIOST/SIOST.kicad_pcb (KiCad board)
At the start: 2 copper layers, 67.3 x 65.5 mm, 11 parts, among them J1 Conn_01x05, J2 Conn_02x23_Odd_Even, J3 Conn_02x23_Odd_Even, J4 Conn_02x07_Odd_Even, J5 Conn_02x16_Odd_Even

Commit message: Cleaned up
Other:
- net class Default removed
- net class Power removed
